File: ESP32_Singlemsg button.kicad_pcb (KiCad board)
At the start: 2 copper layers, 64 x 38 mm, 34 parts, among them J1 Battery, J2 I2C, J3 SPI, J4 USB_C_Receptacle_USB2.0_16P, J5 ANALOG, SW1 RESET, SW2 BOOT, U1 ESP32-S3, U2 AMS1117-3.3, U3 MCP73831-2-OT

Commit message: added silkscreen, ground plane cleaned up interfereing silkscreen note: there is two pullups for en pin drc and erc cleaned up
Routing:
- net D+: track 48.4 -> 44.2 mm
- net SCL: vias 3 -> 2
- net D-: vias 3 -> 2
- added copper zone on B.Cu, net GND
- added copper zone on F.Cu, net GND
Other:
- board text added: "ESP32-S3 BOARD DESIGNED BY AMITH G 14 NOV 2024"
