File: ESP32_Singlemsg button.kicad_sch (KiCad schematic)
At the start: 34 parts, among them J1 Battery, J2 I2C, J3 SPI, J4 USB_C_Receptacle_USB2.0_16P, J5 ANALOG, SW1 RESET, SW2 BOOT, U1 ESP32-S3, U2 AMS1117-3.3, U3 MCP73831-2-OT

Commit message: added silkscreen, ground plane cleaned up interfereing silkscreen note: there is two pullups for en pin drc and erc cleaned up
Connections:
- no-connect marks 0 -> 24
